File: kicad/plate/le_capybara_plate.kicad_sch (KiCad schematic)
At the start: 58 parts, among them SW1 EC_SW

Commit message: getting ready for prototype
Parts:
- added H25, H26, H27, H28, H29, H30, H31, H32, H33, H34, H35, H36, H37, H38: M2 Hole, MountingHole:MountingHole_2.2mm_M2_DIN965, symbol Mechanical:MountingHole
- H1, H10, H11, H12, H13, H14, H15, H16, H17, H18, H19, H2, H20, H21, H22, H23, H24, H3, H4, H5, H6, H7, H8, H9: value MountingHole -> M2 Hole; footprint MountingHole:MountingHole_3.2mm_M3_DIN965 -> MountingHole:MountingHole_2.2mm_M2_DIN965
- SW1: footprint capacitive_sensors:ecs_plate_cut_1U_14x14mm -> capacitive_sensors:ec_plate_cutout_topre_14.1x14.7mm
- SW1: footprint capacitive_sensors:ecs_plate_cut_1U_14x14mm -> capacitive_sensors:ec_plate_cutout_topre_2u

Commit message: Major fixes after prototype order
Fixed the following:
- wrong RGB schematic, D106-D111 doesn't work
- discharge pin from analog circuit was not connected
- plate holes had the wrong diameter
Parts:
- removed H35, H36, H37, H38: M2 Hole, MountingHole:MountingHole_2.2mm_M2_DIN965, symbol Mechanical:MountingHole
- H1, H10, H11, H12, H13, H14, H15, H16, H17, H18, H19, H2, H20, H21, H22, H23, H24, H25, H26, H27, H28, H29, H3, H30, H31, H32, H33, H34, H4, H5, H6, H7, H8, H9: footprint MountingHole:MountingHole_2.2mm_M2_DIN965 -> MountingHole:MountingHole_3.2mm_M3_DIN965

Commit message: schematic fix and plate tolerance fix
Parts:
- H1, H10, H11, H12, H13, H14, H15, H16, H17, H18, H19, H2, H20, H21, H22, H23, H24, H25, H26, H27, H28, H29, H3, H30, H32, H33, H34, H4, H5, H6, H7, H9: footprint MountingHole:MountingHole_3.2mm_M3_DIN965 -> capacitive_sensors:MountingHole_2.2mm_M2
- H31, H8: footprint MountingHole:MountingHole_3.2mm_M3_DIN965 -> capacitive_sensors:MountingHole_2.2mm_M2; now not fitted
- SW1: footprint capacitive_sensors:ec_plate_cutout_topre_14.1x14.7mm -> capacitive_sensors:plate_cut_1U_topre
- SW1: footprint capacitive_sensors:ec_plate_cutout_topre_2u -> capacitive_sensors:plate_cut_2U_topre

Commit message: remove top mounting hole for chiffre+ compatibility
Parts:
- H13, H5: now not fitted
Changed lines of the file:
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@@
   )
   (symbol (lib_id "Mechanical:MountingHole") (at 38.1 116.84 0) (unit 1)
-    (in_bom yes) (on_board yes) (dnp no) (fields_autoplaced)
+    (in_bom yes) (on_board yes) (dnp yes) (fields_autoplaced)
     (property "Reference" "H5" (at 40.64 115.57 0)
       (effects (font (size 1.27 1.27)) (justify left))
@@
   )
   (symbol (lib_id "Mechanical:MountingHole") (at 38.1 132.08 0) (unit 1)
-    (in_bom yes) (on_board yes) (dnp no) (fields_autoplaced)
+    (in_bom yes) (on_board yes) (dnp yes) (fields_autoplaced)
     (property "Reference" "H13" (at 40.64 130.81 0)
       (effects (font (size 1.27 1.27)) (justify left))
