File: kicad/plate_36keys/plate_36keys.kicad_pcb (KiCad board)
At the start: 2 copper layers, 231.6 x 92.5 mm, 53 parts, among them SW1 EC_SW, SW10 EC_SW, SW11 EC_SW, SW12 EC_SW, SW13 EC_SW, SW14 EC_SW, SW15 EC_SW, SW16 EC_SW, SW17 EC_SW, SW18 EC_SW, SW19 EC_SW, SW2 EC_SW, SW20 EC_SW, SW21 EC_SW, SW22 EC_SW, SW23 EC_SW, SW24 EC_SW, SW25 EC_SW, SW26 EC_SW, SW27 EC_SW, SW28 EC_SW, SW29 EC_SW, SW3 EC_SW, SW30 EC_SW, SW31 EC_SW, SW32 EC_SW, SW33 EC_SW, SW34 EC_SW, SW35 EC_SW, SW4 EC_SW, SW5 EC_SW, SW6 EC_SW, SW7 EC_SW, SW8 EC_SW, SW9 EC_SW

Commit message: Production plates - all versions
Parts:
- added SW36: EC_SW, capacitive_sensors:plate_cut_1U_topre, F.Cu at (220.5, 130.7)
- SW33: footprint capacitive_sensors:plate_cut_2U_topre -> capacitive_sensors:plate_cut_1U_topre
- moved SW34 16.7 mm to (201.6, 133.0)
- moved SW33 7.14 mm to (180.3, 135.6)
- moved H16 2.38 mm to (211.0, 131.8)
Other:
- board text added: "Le Capybara Plate 36-keys"
- board text removed: "Le Capybara Plate Asymmetric"
