File: kicad/pcb/key_matrix.kicad_sch (KiCad schematic)
At the start: 38 parts, among them SW1 EC_SW, SW10 EC_SW, SW11 EC_SW, SW12 EC_SW, SW13 EC_SW, SW14 EC_SW, SW15 EC_SW, SW2 EC_SW, SW3 EC_SW, SW35 SW_Push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

Commit message: rerouted pcb
Connections:
- net COL0: now also SW1.1, SW2.1, SW3.1; no longer SW1.2, SW2.2, SW3.2
- net COL1: now also SW4.1, SW5.1, SW6.1; no longer SW4.2, SW5.2, SW6.2
- net COL2: now also SW3.1, SW7.1, SW8.1, SW9.1; no longer SW3.2, SW7.2, SW8.2, SW9.2
- net COL3: now also SW10.1, SW11.1, SW12.1; no longer SW10.2, SW11.2, SW12.2
- net COL4: now also SW13.1, SW14.1, SW15.1; no longer SW13.2, SW14.2, SW15.2
- net COL5: now also SW14.2; no longer SW14.1
- net ROW0: now also SW1.2, SW10.2, SW13.2, SW4.2, SW7.2; no longer SW1.1, SW10.1, SW13.1, SW4.1, SW7.1
- net ROW1: now also SW11.2, SW14.1, SW14.2, SW2.2, SW5.2, SW8.2; no longer SW11.1, SW14.1, SW14.2, SW2.1, SW5.1, SW8.1
- net ROW2: now also SW12.2, SW15.2, SW3.2, SW6.2, SW9.2; no longer SW12.1, SW15.1, SW3.1, SW6.1, SW9.1
- net ROW3: now also SW3.2; no longer SW3.1
Changed lines of the file:
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@@
     )
   )
-  (symbol (lib_id "cipulot_parts:EC_SW") (at 133.985 39.37 0) (mirror y) (unit 1)
+  (symbol (lib_id "cipulot_parts:EC_SW") (at 133.985 39.37 0) (unit 1)
     (in_bom no) (on_board yes) (dnp no)
     (property "Reference" "SW13" (at 133.985 33.02 0)
@@
     )
   )
-  (symbol (lib_id "cipulot_parts:EC_SW") (at 133.985 58.42 0) (mirror y) (unit 1)
+  (symbol (lib_id "cipulot_parts:EC_SW") (at 133.985 58.42 0) (unit 1)
     (in_bom no) (on_board yes) (dnp no)
     (property "Reference" "SW14" (at 133.985 52.07 0)
@@
     )
   )
-  (symbol (lib_id "cipulot_parts:EC_SW") (at 65.405 58.42 0) (mirror y) (unit 1)
+  (symbol (lib_id "cipulot_parts:EC_SW") (at 65.405 58.42 0) (unit 1)
     (in_bom no) (on_board yes) (dnp no)
     (property "Reference" "SW5" (at 65.405 52.07 0)
@@
     )
   )
-  (symbol (lib_id "cipulot_parts:EC_SW") (at 88.265 77.47 0) (mirror y) (unit 1)
+  (symbol (lib_id "cipulot_parts:EC_SW") (at 88.265 77.47 0) (unit 1)
     (in_bom no) (on_board yes) (dnp no)
     (property "Reference" "SW9" (at 88.265 71.12 0)
@@
     )
   )
-  (symbol (lib_id "cipulot_parts:EC_SW") (at 88.265 58.42 0) (mirror y) (unit 1)
+  (symbol (lib_id "cipulot_parts:EC_SW") (at 88.265 58.42 0) (unit 1)
     (in_bom no) (on_board yes) (dnp no)
     (property "Reference" "SW8" (at 88.265 52.07 0)
@@
     )
   )
-  (symbol (lib_id "cipulot_parts:EC_SW") (at 88.265 96.52 0) (mirror y) (unit 1)
+  (symbol (lib_id "cipulot_parts:EC_SW") (at 88.265 96.52 0) (unit 1)
     (in_bom no) (on_board yes) (dnp no)
     (property "Reference" "SW3" (at 88.265 90.17 0)
@@
     )
   )
-  (symbol (lib_id "cipulot_parts:EC_SW") (at 111.125 58.42 0) (mirror y) (unit 1)
+  (symbol (lib_id "cipulot_parts:EC_SW") (at 111.125 58.42 0) (unit 1)
     (in_bom no) (on_board yes) (dnp no)
     (property "Reference" "SW11" (at 111.125 52.07 0)
@@
     )
   )
-  (symbol (lib_id "cipulot_parts:EC_SW") (at 88.265 39.37 0) (mirror y) (unit 1)
+  (symbol (lib_id "cipulot_parts:EC_SW") (at 88.265 39.37 0) (unit 1)
     (in_bom no) (on_board yes) (dnp no)
     (property "Reference" "SW7" (at 88.265 33.02 0)
@@
     )
   )
-  (symbol (lib_id "cipulot_parts:EC_SW") (at 42.545 77.47 0) (mirror y) (unit 1)
+  (symbol (lib_id "cipulot_parts:EC_SW") (at 42.545 77.47 0) (unit 1)
     (in_bom no) (on_board yes) (dnp no)
     (property "Reference" "SW3" (at 42.545 71.12 0)
@@
     )
   )
-  (symbol (lib_id "cipulot_parts:EC_SW") (at 168.275 58.42 0) (mirror y) (unit 1)
+  (symbol (lib_id "cipulot_parts:EC_SW") (at 168.275 58.42 0) (unit 1)
     (in_bom no) (on_board yes) (dnp no)
     (property "Reference" "SW14" (at 168.275 52.07 0)
@@
     )
   )
-  (symbol (lib_id "cipulot_parts:EC_SW") (at 65.405 39.37 0) (mirror y) (unit 1)
+  (symbol (lib_id "cipulot_parts:EC_SW") (at 65.405 39.37 0) (unit 1)
     (in_bom no) (on_board yes) (dnp no)
     (property "Reference" "SW4" (at 65.405 33.02 0)
@@
     )
   )
-  (symbol (lib_id "cipulot_parts:EC_SW") (at 133.985 77.47 0) (mirror y) (unit 1)
+  (symbol (lib_id "cipulot_parts:EC_SW") (at 133.985 77.47 0) (unit 1)
     (in_bom no) (on_board yes) (dnp no)
     (property "Reference" "SW15" (at 133.985 71.12 0)
@@
     )
   )
-  (symbol (lib_id "cipulot_parts:EC_SW") (at 42.545 39.37 0) (mirror y) (unit 1)
+  (symbol (lib_id "cipulot_parts:EC_SW") (at 42.545 39.37 0) (unit 1)
     (in_bom no) (on_board yes) (dnp no)
     (property "Reference" "SW1" (at 42.545 33.02 0)
@@
     )
   )
-  (symbol (lib_id "cipulot_parts:EC_SW") (at 42.545 58.42 0) (mirror y) (unit 1)
+  (symbol (lib_id "cipulot_parts:EC_SW") (at 42.545 58.42 0) (unit 1)
     (in_bom no) (on_board yes) (dnp no)
     (property "Reference" "SW2" (at 42.545 52.07 0)
@@
     )
   )
-  (symbol (lib_id "cipulot_parts:EC_SW") (at 111.125 77.47 0) (mirror y) (unit 1)
+  (symbol (lib_id "cipulot_parts:EC_SW") (at 111.125 77.47 0) (unit 1)
     (in_bom no) (on_board yes) (dnp no)
     (property "Reference" "SW12" (at 111.125 71.12 0)
@@
     )
   )
-  (symbol (lib_id "cipulot_parts:EC_SW") (at 111.125 39.37 0) (mirror y) (unit 1)
+  (symbol (lib_id "cipulot_parts:EC_SW") (at 111.125 39.37 0) (unit 1)
     (in_bom no) (on_board yes) (dnp no)
     (property "Reference" "SW10" (at 111.125 33.02 0)
@@
     )
   )
-  (symbol (lib_id "cipulot_parts:EC_SW") (at 65.405 77.47 0) (mirror y) (unit 1)
+  (symbol (lib_id "cipulot_parts:EC_SW") (at 65.405 77.47 0) (unit 1)
     (in_bom no) (on_board yes) (dnp no)
     (property "Reference" "SW6" (at 65.405 71.12 0)

Commit message: getting ready for prototype
Parts:
- added SW3 (x6): EC_SW, capacitive_sensors:ec_pad_1U_90deg, symbol cipulot_parts:EC_SW
- SW3: footprint capacitive_sensors:capy_pad_1U_90deg -> capacitive_sensors:ec_pad_1U_90deg
- SW35: footprint modified_footrprints:MX-Solderable-1U -> modified_footprints:MX-Solderable-1U
- SW36: footprint modified_footrprints:ROT_Alps_EC11E-Switch -> modified_footprints:ROT_Alps_EC11E-Switch
Connections:
- net COL1: now also SW3.1, SW3.1
- net COL2: now also SW3.2; no longer SW3.1
- net COL3: now also SW3.2
- net COL6: now also SW3.2
- net COL7: now also SW3.2; no longer SW3.1
- net COL8: now also SW3.1, SW3.1
- net GND: now also SW3.3 (SG), SW3.3 (SG), SW3.3 (SG), SW3.3 (SG), SW3.3 (SG), SW3.3 (SG)
- net ROW3: now also SW3.1, SW3.1, SW3.1, SW3.1, SW3.2, SW3.2
Other:
- moved on the sheet: C18, C19, SW3, SW35, SW36

Commit message: schematic fix and plate tolerance fix
Parts:
- removed SW3 (x2): EC_SW, capacitive_sensors:ec_pad_1U_90deg, symbol cipulot_parts:EC_SW
- SW3: footprint capacitive_sensors:ec_pad_1U_90deg -> capacitive_sensors:capy_pad_2U_90deg
- SW3: footprint capacitive_sensors:ec_pad_1U_90deg -> capacitive_sensors:ecs_pad_combo_0.125u_offset
Connections:
- net COL1: now also SW3.2; no longer SW3.1
- net ROW3: now also SW3.1; no longer SW3.2
Changed lines of the file:
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@@
   (junction (at 150.495 44.45) (diameter 0) (color 0 0 0 0)
   )
-  (junction (at 182.88 157.48) (diameter 0) (color 0 0 0 0)
-  )
   (junction (at 88.265 82.55) (diameter 0) (color 0 0 0 0)
   )
@@
   (junction (at 42.926 124.841) (diameter 0) (color 0 0 0 0)
   )
-  (junction (at 175.26 152.4) (diameter 0) (color 0 0 0 0)
-  )
   (junction (at 111.125 44.45) (diameter 0) (color 0 0 0 0)
   )
@@
   (junction (at 236.855 82.55) (diameter 0) (color 0 0 0 0)
   )
-  (junction (at 241.3 157.48) (diameter 0) (color 0 0 0 0)
-  )
   (junction (at 175.895 39.37) (diameter 0) (color 0 0 0 0)
   )
   (junction (at 57.785 58.42) (diameter 0) (color 0 0 0 0)
   )
-  (junction (at 231.14 152.4) (diameter 0) (color 0 0 0 0)
-  )
   (junction (at 229.235 48.26) (diameter 0) (color 0 0 0 0)
   )
@@
     (stroke (width 0) (type default))
   )
-  (wire (pts (xy 149.86 137.16) (xy 149.86 147.32))
-    (stroke (width 0) (type default))
-  )
   (wire (pts (xy 42.926 124.841) (xy 60.706 124.841))
     (stroke (width 0) (type default))
@@
     (stroke (width 0) (type default))
   )
-  (wire (pts (xy 248.92 157.48) (xy 241.3 157.48))
-    (stroke (width 0) (type default))
-  )
   (wire (pts (xy 87.376 127.381) (xy 104.521 127.381))
     (stroke (width 0) (type default))
@@
     (stroke (width 0) (type default))
   )
-  (wire (pts (xy 248.92 152.4) (xy 231.14 152.4))
-    (stroke (width 0) (type default))
-  )
-  (wire (pts (xy 241.3 147.32) (xy 241.3 157.48))
-    (stroke (width 0) (type default))
-  )
   (wire (pts (xy 80.391 135.001) (xy 80.391 129.921))
     (stroke (width 0) (type default))
@@
     (stroke (width 0) (type default))
   )
-  (wire (pts (xy 256.54 137.16) (xy 256.54 147.32))
-    (stroke (width 0) (type default))
-  )
   (wire (pts (xy 118.745 58.42) (xy 118.745 67.31))
     (stroke (width 0) (type default))
@@
     (stroke (width 0) (type default))
   )
-  (wire (pts (xy 157.48 152.4) (xy 175.26 152.4))
-    (stroke (width 0) (type default))
-  )
   (wire (pts (xy 42.926 135.636) (xy 42.926 136.906))
     (stroke (width 0) (type default))
@@
     (stroke (width 0) (type default))
   )
-  (wire (pts (xy 165.1 157.48) (xy 182.88 157.48))
-    (stroke (width 0) (type default))
-  )
   (wire (pts (xy 65.405 63.5) (xy 88.265 63.5))
     (stroke (width 0) (type default))
@@
     (stroke (width 0) (type default))
   )
-  (wire (pts (xy 165.1 147.32) (xy 165.1 157.48))
-    (stroke (width 0) (type default))
-  )
   (wire (pts (xy 231.14 152.4) (xy 213.36 152.4))
     (stroke (width 0) (type default))
@@
     (stroke (width 0) (type default))
   )
-  (wire (pts (xy 223.52 157.48) (xy 241.3 157.48))
+  (wire (pts (xy 223.52 157.48) (xy 248.92 157.48))
     (stroke (width 0) (type default))
   )
@@
     (effects (font (size 1.27 1.27)) (justify left))
     (property "Intersheetrefs" "${INTERSHEET_REFS}" (at 280.5822 86.36 0)
-      (effects (font (size 1.27 1.27)) (justify left) hide)
-    )
-  )
-  (global_label "COL8" (shape input) (at 256.54 137.16 90) (fields_autoplaced)
-    (effects (font (size 1.27 1.27)) (justify left))
-    (property "Intersheetrefs" "${INTERSHEET_REFS}" (at 256.54 129.4161 90)
       (effects (font (size 1.27 1.27)) (justify left) hide)
     )
@@
     )
   )
-  (global_label "COL1" (shape input) (at 149.86 137.16 90) (fields_autoplaced)
-    (effects (font (size 1.27 1.27)) (justify left))
-    (property "Intersheetrefs" "${INTERSHEET_REFS}" (at 149.86 129.4161 90)
-      (effects (font (size 1.27 1.27)) (justify left) hide)
-    )
-  )
   (global_label "COL3" (shape input) (at 103.505 31.75 90) (fields_autoplaced)
     (effects (font (size 1.27 1.27)) (justify left))
@@
       (effects (font (size 1.27 1.27)))
     )
-    (property "Footprint" "capacitive_sensors:ec_pad_1U_90deg" (at 191.135 96.52 0)
+    (property "Footprint" "capacitive_sensors:capy_pad_2U_90deg" (at 191.135 96.52 0)
       (effects (font (size 1.27 1.27)) hide)
     )
@@
     )
   )
-  (symbol (lib_id "cipulot_parts:EC_SW") (at 65.405 96.52 0) (unit 1)
+  (symbol (lib_id "cipulot_parts:EC_SW") (at 65.405 96.52 0) (mirror y) (unit 1)
     (in_bom no) (on_board yes) (dnp no)
     (property "Reference" "SW3" (at 65.405 90.17 0)
@@
       (effects (font (size 1.27 1.27)))
     )
-    (property "Footprint" "capacitive_sensors:ec_pad_1U_90deg" (at 65.405 96.52 0)
+    (property "Footprint" "capacitive_sensors:ecs_pad_combo_0.125u_offset" (at 65.405 96.52 0)
       (effects (font (size 1.27 1.27)) hide)
     )
@@
       (effects (font (size 1.27 1.27)))
     )
-    (property "Footprint" "capacitive_sensors:ec_pad_1U_90deg" (at 111.125 96.52 0)
+    (property "Footprint" "capacitive_sensors:capy_pad_2U_90deg" (at 111.125 96.52 0)
       (effects (font (size 1.27 1.27)) hide)
     )
@@
     )
   )
-  (symbol (lib_id "cipulot_parts:EC_SW") (at 157.48 147.32 0) (unit 1)
-    (in_bom no) (on_board yes) (dnp no)
-    (property "Reference" "SW3" (at 157.48 140.97 0)
-      (effects (font (size 1.27 1.27)))
-    )
-    (property "Value" "EC_SW" (at 157.48 143.51 0)
-      (effects (font (size 1.27 1.27)))
-    )
-    (property "Footprint" "capacitive_sensors:ec_pad_1U_90deg" (at 157.48 147.32 0)
-      (effects (font (size 1.27 1.27)) hide)
-    )
-    (property "Datasheet" "" (at 157.48 147.32 0)
-      (effects (font (size 1.27 1.27)))
-    )
-    (pin "1")
-    (pin "2")
-    (pin "3")
-    (instances
-      (project "tako"
-        (path "/7b28ce14-5c63-4c9f-9bca-abf529f54075"
-          (reference "SW3") (unit 1)
-        )
-      )
-      (project "tako"
-        (path "/9d8265e2-df3b-4900-a886-1f487fd3d916"
-          (reference "SW16") (unit 1)
-        )
-      )
-      (project "le_capybara"
-        (path "/ca0d59d2-7f9b-4344-99bc-39bc2c8c88cb/9412d715-f7b7-4535-9cc7-549a2178ec10"
-          (reference "SW38") (unit 1)
-        )
-      )
-    )
-  )
   (symbol (lib_id "cipulot_parts:EC_SW") (at 168.275 58.42 0) (unit 1)
     (in_bom no) (on_board yes) (dnp no)
@@
       (effects (font (size 1.27 1.27)))
     )
-    (property "Footprint" "capacitive_sensors:ec_pad_1U_90deg" (at 236.855 96.52 0)
+    (property "Footprint" "capacitive_sensors:ecs_pad_combo_0.125u_offset" (at 236.855 96.52 0)
       (effects (font (size 1.27 1.27)) hide)
     )
@@
         )
       )
-    )
-  )
-  (symbol (lib_id "cipulot_parts:EC_SW") (at 248.92 147.32 0) (mirror y) (unit 1)
-    (in_bom no) (on_board yes) (dnp no)
-    (property "Reference" "SW3" (at 248.92 140.97 0)
-      (effects (font (size 1.27 1.27)))
-    )
-    (property "Value" "EC_SW" (at 248.92 143.51 0)
-      (effects (font (size 1.27 1.27)))
-    )
-    (property "Footprint" "capacitive_sensors:ec_pad_1U_90deg" (at 248.92 147.32 0)
-      (effects (font (size 1.27 1.27)) hide)
-    )
-    (property "Datasheet" "" (at 248.92 147.32 0)
-      (effects (font (size 1.27 1.27)))
-    )
-    (pin "1")
-    (pin "2")
-    (pin "3")
-    (instances
-      (project "tako"
-        (path "/7b28ce14-5c63-4c9f-9bca-abf529f54075"
-          (reference "SW3") (unit 1)
-        )
-      )
-      (project "tako"
-        (path "/9d8265e2-df3b-4900-a886-1f487fd3d916"
-          (reference "SW16") (unit 1)
-        )
-      )
-      (project "le_capybara"
-        (path "/ca0d59d2-7f9b-4344-99bc-39bc2c8c88cb/9412d715-f7b7-4535-9cc7-549a2178ec10"
-          (reference "SW41") (unit 1)
-        )
-      )
