File: kicad/plate_asym/plate_asym.kicad_pcb (KiCad board)
At the start: 2 copper layers, 231.6 x 92.5 mm, 51 parts, among them SW1 EC_SW, SW10 EC_SW, SW11 EC_SW, SW12 EC_SW, SW13 EC_SW, SW14 EC_SW, SW15 EC_SW, SW16 EC_SW, SW17 EC_SW, SW18 EC_SW, SW19 EC_SW, SW2 EC_SW, SW20 EC_SW, SW21 EC_SW, SW22 EC_SW, SW23 EC_SW, SW24 EC_SW, SW25 EC_SW, SW26 EC_SW, SW27 EC_SW, SW28 EC_SW, SW29 EC_SW, SW3 EC_SW, SW30 EC_SW, SW31 EC_SW, SW32 EC_SW, SW33 EC_SW, SW34 EC_SW, SW35 EC_SW, SW4 EC_SW, SW5 EC_SW, SW6 EC_SW, SW7 EC_SW, SW8 EC_SW, SW9 EC_SW

Commit message: Remove extra mounting holes from PCB and update version number.
Other:
- board text added: "Le Capybara Plate (Asymmetric)"
- board text removed: "Le Capybara Plate Asymmetric"
Changed lines of the file:
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@@
   (title_block
     (title "Le Capybara")
-    (date "2023-07-07")
-    (rev "v0.1")
+    (date "2024-02-21")
+    (rev "1.0")
     (company "sporkus")
   )
@@
     (effects (font (size 2 2) (thickness 0.3)) (justify left bottom))
   )
-  (gr_text "Le Capybara Plate Asymmetric" (at 39.880343 56.647143) (layer "User.1")
+  (gr_text "Le Capybara Plate (Asymmetric)" (at 39.880343 56.647143) (layer "User.1")
     (effects (font (size 4 4) (thickness 0.3)) (justify left bottom))
   )
@@
     (effects (font (size 2 2) (thickness 0.3)) (justify left bottom))
   )
-  (gr_text_box "Drill notes:\n\nA = 16 x M2x0.4mm threaded\nB = 8 x ⌀2.2mm THRU"
+  (gr_text_box "Material thickness: 1.2mm\n\nDrill notes:\n\nA = 16 x M2x0.4mm threaded\nB = 8 x ⌀2.2mm THRU"
     (start 221.917843 143.497143) (end 273.242843 164.897143) (layer "User.1")
       (effects (font (size 2 2) (thickness 0.2)) (justify left top))
